File: MAX485.kicad_sch (KiCad schematic)
At the start: 11 parts, among them U2 MAX485E

Commit message: Add files via upload
Connections:
- net +5V: now also C3.1; no longer C3.2
- net GND: now also C3.2; no longer C3.1
Other:
- moved on the sheet: C3
Changed lines of the file:
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@@
 	(symbol
 		(lib_id "Device:C")
-		(at 153.67 77.47 90)
+		(at 153.67 77.47 270)
 		(unit 1)
 		(exclude_from_sim no)
@@
 		)
 		(property "Footprint" "inqbe:CP_Radial_D5.0mm_P2.50mm"
-			(at 157.48 76.5048 0)
+			(at 149.86 78.4352 0)
 			(effects
 				(font
