File: servo_diff_to_single.kicad_pcb (KiCad board)
At the start: 2 copper layers, 128.3 x 91.4 mm, 77 parts, among them J1 Barrel_Jack_Switch, J2 DE15_Receptacle_HighDensity, J3 Conn_02x05_Odd_Even, J4 Conn_01x05_Socket, U1 LM7805_TO220, U2 MAX485E, U3 MAX485E, U4 MAX485E, U5 MAX485E, U6 MAX485E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

Commit message: Add files via upload
Parts:
- moved C4 2.77 mm to (109.9, 63.5), turned to 0 degrees
- moved C1 2.54 mm to (143.5, 120.0), turned to 0 degrees
- moved C5 2.54 mm to (109.2, 88.9), turned to 0 degrees
- moved C3 2.54 mm to (66.0, 63.5), turned to 0 degrees
- moved C7 2.48 mm to (109.9, 114.3), turned to 0 degrees
- moved C8 2.48 mm to (66.1, 114.3), turned to 0 degrees
- moved C6 2.45 mm to (66.1, 88.9), turned to 0 degrees
- moved C2 2.41 mm to (132.1, 133.3), turned to 90 degrees
Connections:
- C1 pad 1: GND -> Net-(U1-VI)
- C1 pad 2: Net-(U1-VI) -> GND
- C2 pad 1: GND -> +5V
- C2 pad 2: +5V -> GND
- C3 pad 1: GND -> +5V
- C3 pad 2: +5V -> GND
- C4 pad 1: GND -> +5V
- C4 pad 2: +5V -> GND
- C5 pad 1: GND -> +5V
- C5 pad 2: +5V -> GND
- C6 pad 1: GND -> +5V
- C6 pad 2: +5V -> GND
- C7 pad 1: GND -> +5V
- C7 pad 2: +5V -> GND
- C8 pad 1: GND -> +5V
- C8 pad 2: +5V -> GND
