File: servo_diff_to_single.kicad_sch (KiCad schematic)
At the start: 7 parts, among them J1 Barrel_Jack_Switch, J2 DE15_Receptacle_HighDensity, J3 Conn_02x05_Odd_Even, J4 Conn_01x05_Socket, U1 LM7805_TO220

Commit message: Add files via upload
Connections:
- net +5V: now also C2.1; no longer C2.2
- net GND: now also C1.2, C2.2; no longer C1.1, C2.1
- net at J1.1, U1.1 (VI): now also C1.1; no longer C1.2
Other:
- moved on the sheet: C1, C2
